Commit message: add imu plugin to mid360 model

File: urdf/livox_mid360.xacro (robot description, xacro)
@@ -58,4 +58,17 @@
     </gazebo>
   </xacro:macro>
+  <xacro:macro name="Livox_Mid_gazebo_imu" params="name:=livox">
+    <gazebo>
+      <plugin name="imu_plugin" filename="libgazebo_ros_imu.so">
+        <bodyName>${name}_base</bodyName>
+        <robotNamespace>${name}</robotNamespace>
+        <topicName>imu</topicName>
+        <serviceName>imu_service</serviceName>
+        <gaussianNoise>0.01</gaussianNoise>
+        <updateRate>200.0</updateRate>
+        <alwaysOn>true</alwaysOn>
+      </plugin>
+    </gazebo>
+  </xacro:macro>
   <xacro:macro name="Livox_Mid40" params="visualize:=True name:=livox">
     <link name="${name}_base">
@@ -83,4 +96,5 @@
     </joint>
     <xacro:Livox_Mid_gazebo_sensor name="${name}" visualize="${visualize}"/>
+    <xacro:Livox_Mid_gazebo_imu name="${name}"/>
   </xacro:macro>
     <xacro:Livox_Mid40 name="livox"/>

Commit message: changed rostopic name

File: urdf/livox_mid360.xacro (robot description, xacro)
@@ -4,5 +4,5 @@
   <xacro:property name="laser_min_range" value="0.1"/>
   <xacro:property name="laser_max_range" value="200.0"/>
-  <xacro:property name="ros_topic" value="scan"/>
+  <xacro:property name="ros_topic" value="lidar"/>
   <xacro:property name="samples" value="24000"/>
   <xacro:property name="downsample" value="1"/>
@@ -53,5 +53,5 @@
 		  <downsample>${downsample}</downsample>
 		  <csv_file_name>package://livox_laser_simulation/scan_mode/mid360.csv</csv_file_name>
-		  <ros_topic>${ros_topic}</ros_topic>
+		  <ros_topic>${name}/${ros_topic}</ros_topic>
         </plugin>
       </sensor>

Commit message: use libgazebo_ros_imu_sensor.so and refactored urdf

File: urdf/livox_mid360.xacro (robot description, xacro)
@@ -10,7 +10,7 @@
     <inertial>
       <mass value="0.1"/>
-    <inertia ixx="0.01" ixy="0" ixz="0"
-          iyy="0.01" iyz="0"
-          izz="0.01"/>
+      <inertia ixx="0.01" ixy="0" ixz="0"
+               iyy="0.01" iyz="0"
+               izz="0.01"/>
     </inertial>
   </xacro:macro>
@@ -23,35 +23,35 @@
         <!-- This ray plgin is only for visualization. -->
         <plugin name="gazebo_ros_laser_controller" filename="liblivox_laser_simulation.so">
-			<ray>
-			  <scan>
-				<horizontal>
-				<samples>100</samples>
-				<resolution>1</resolution>
-				<min_angle>${0}</min_angle>
-				<max_angle>${2*M_PI}</max_angle>
-				</horizontal>
-				<vertical>
-				<samples>360</samples>
-				<resolution>1</resolution>
-				<min_angle>${-7.22/180*M_PI}</min_angle>
-				<max_angle>${55.22/180*M_PI}</max_angle>
-				</vertical>
-			  </scan>
-			  <range>
-				<min>${laser_min_range}</min>
-				<max>${laser_max_range}</max>
-				<resolution>${resolution}</resolution>
-			  </range>
-			  <noise>
-				<type>gaussian</type>
-				<mean>${noise_mean}</mean>
-				<stddev>${noise_stddev}</stddev>
-			  </noise>
-			</ray>
+          <ray>
+            <scan>
+              <horizontal>
+                <samples>100</samples>
+                <resolution>1</resolution>
+                <min_angle>${0}</min_angle>
+                <max_angle>${2*M_PI}</max_angle>
+              </horizontal>
+              <vertical>
+                <samples>360</samples>
+                <resolution>1</resolution>
+                <min_angle>${-7.22/180*M_PI}</min_angle>
+                <max_angle>${55.22/180*M_PI}</max_angle>
+              </vertical>
+            </scan>
+            <range>
+              <min>${laser_min_range}</min>
+              <max>${laser_max_range}</max>
+              <resolution>${resolution}</resolution>
+            </range>
+            <noise>
+              <type>gaussian</type>
+              <mean>${noise_mean}</mean>
+              <stddev>${noise_stddev}</stddev>
+            </noise>
+          </ray>
           <visualize>${visualize}</visualize>
-		  <samples>${samples}</samples>
-		  <downsample>${downsample}</downsample>
-		  <csv_file_name>package://livox_laser_simulation/scan_mode/mid360.csv</csv_file_name>
-		  <ros_topic>${name}/${ros_topic}</ros_topic>
+          <samples>${samples}</samples>
+          <downsample>${downsample}</downsample>
+          <csv_file_name>package://livox_laser_simulation/scan_mode/mid360.csv</csv_file_name>
+          <ros_topic>${name}/${ros_topic}</ros_topic>
         </plugin>
       </sensor>
@@ -59,14 +59,21 @@
   </xacro:macro>
   <xacro:macro name="Livox_Mid_gazebo_imu" params="name:=livox">
-    <gazebo>
-      <plugin name="imu_plugin" filename="libgazebo_ros_imu.so">
-        <bodyName>${name}_base</bodyName>
-        <robotNamespace>${name}</robotNamespace>
-        <topicName>imu</topicName>
-        <serviceName>imu_service</serviceName>
-        <gaussianNoise>0.01</gaussianNoise>
-        <updateRate>200.0</updateRate>
-        <alwaysOn>true</alwaysOn>
-      </plugin>
+    <gazebo reference="${name}">
+      <sensor type="imu" name="${name}_imu">
+        <pose>0 0 0 0 0 0</pose>
+        <update_rate>200</update_rate>
+        <plugin name="imu_plugin" filename="libgazebo_ros_imu_sensor.so">
+          <frameName>laser_livox</frameName>
+          <robotNamespace>${name}</robotNamespace>
+          <topicName>imu</topicName>
+          <serviceName>imu_service</serviceName>
+          <gaussianNoise>0.01</gaussianNoise>
+          <updateRateHZ>1000</updateRateHZ>
+          <xyzOffset>0 0 0</xyzOffset>
+          <rpyOffset>0 0 0</rpyOffset>
+          <alwaysOn>true</alwaysOn>
+          <initialOrientationAsReference>false</initialOrientationAsReference>
+        </plugin>
+      </sensor>
     </gazebo>
   </xacro:macro>
@@ -82,7 +89,8 @@
       </visual>
       <collision>
-		  <origin xyz="0 0 0" rpy="0 0 0" /> <geometry> <mesh
-		  filename="package://livox_laser_simulation/meshes/livox_mid40.dae">
-		  </mesh> </geometry>
+        <origin xyz="0 0 0" rpy="0 0 0" />
+        <geometry>
+          <mesh filename="package://livox_laser_simulation/meshes/livox_mid40.dae"/>
+        </geometry>
       </collision>
     </link>
@@ -98,5 +106,5 @@
     <xacro:Livox_Mid_gazebo_imu name="${name}"/>
   </xacro:macro>
-    <xacro:Livox_Mid40 name="livox"/>
+  <xacro:Livox_Mid40 name="livox"/>
   <xacro:include filename="$(find livox_laser_simulation)/urdf/standardrobots_oasis300.xacro"/>
   <xacro:link_oasis name="oasis"/>
